Commit message: Grasper assembly

File: manipulador_description/urdf/manipulador.urdf (robot description, URDF)
Before this commit: robot manipulador, 7 links, 6 joints
Links:
- link Grasper: geometry collision mesh filename=package://manipulador_description/Grasper/GrasperBody.stl; collision mesh filename=package://manipulador_description/meshes/Grasper/Grasper1.s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
Joints:
- joint fourth: origin xyz=1.826 -0.001 0.17 rpy=0 0 0 -> xyz=1.826 0 0.17 rpy=0 0 0
- joint second: origin xyz=0.116 -0.015 0.85 rpy=0 0 0 -> xyz=0.116 0 0.85 rpy=0 0 0
- joint third: origin xyz=0.001 0.014 1.6 rpy=0 0 0 -> xyz=0 0 1.6 rpy=0 0 0

Commit message: coliision position

File: manipulador_description/urdf/manipulador.urdf (robot description, URDF)
Before this commit: robot manipulador, 7 links, 6 joints
Links:
- removed link floor
- added link world
- link Grasper: geometry visual mesh filename=package://manipulador_description/meshes/Grasper/GrasperBod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
Joints:
- removed joint base
- added joint world_joint: type fixed, parent world, child Support, origin xyz=0.0 0.0 0.0 rpy=0.0 0.0 0.0

File: manipulador_description/urdf/parts.urdf (robot description, URDF)
Before this commit: robot manipulador, 7 links, 6 joints
Links:
- link Grasper: geometry collision mesh filename=package://manipulador_description/Grasper/GrasperBody.stl; collision mesh filename=package://manipulador_description/meshes/Grasper/Grasper1.s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

Commit message: fifth joint PID

File: manipulador_description/urdf/manipulador.urdf (robot description, URDF)
Before this commit: robot manipulador, 7 links, 6 joints
Links:
- link Grasper: geometry collision cylinder length=0.7 radius=0.04; visual cylinder length=0.7 radius=0.04
Joints:
- joint fifth: limit lower=-1.5708 upper=1.5708 effort=50 velocity=1 -> lower=-1.5708 upper=0 effort=50 velocity=1; origin xyz=0 0 -0.37 rpy=0 0 0 -> xyz=0 0 -0.6 rpy=0 0 0

Commit message: update

File: manipulador_description/urdf/manipulador.urdf (robot description, URDF)
Before this commit: robot manipulador, 7 links, 6 joints
Links:
- link Base: mass 1.0 -> 0.791
- link Grasper: mass 0.1 -> 0.03; geometry collision mesh filename=package://manipulador_description/meshes/Grasper/GrasperBod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; visual mesh filename=package://manipulador_description/meshes/Grasper/GrasperBod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
- link GrasperHolder: mass 0.1 -> 0.068
- link LowerArm: mass 1.0 -> 0.464
- link Support: mass 1.0 -> 0.73
- link UpperArm: mass 0.2 -> 0.407
Joints:
- joint fifth: origin xyz=0 0 -0.6 rpy=0 0 0 -> xyz=0 0 -0.37 rpy=0 0 0

File: manipulador_description/urdf/manipulador.xacro (robot description, xacro)
@@ -3,3 +3,4 @@
 	<!-- Put here the robot description -->
 	<xacro:include filename="$(find manipulador_description)/urdf/manipulador.urdf" />
+	<xacro:include filename="$(find manipulador_description)/urdf/materials.xacro" />
 </robot>
